File: SwiftFi.kicad_sch (KiCad schematic)
At the start: 29 parts, among them J1 Addl Signals, J2 Programming, Q1 BSS138, Q2 BSS138, Q3 BSS138, Q4 BSS138, Q5 BSS138, U1 6526, U2 6551, U3 74HC74, U4 ESP-12E, U5 LM1117-3.3, Y1 3.6864 MHz

Commit message: changed footprints caps, added llinks to aliexpress in BOM
Parts:
- C1, C2: footprint Capacitor_Tantalum_SMD:CP_EIA-2012-12_Kemet-R_Pad1.30x1.05mm_HandSolder -> Capacitor_Tantalum_SMD:CP_EIA-3216-10_Kemet-I_Pad1.58x1.35mm_HandSolder; AliExpress (none) -> https://www.aliexpress.com/item/1005002349845549.html
- C3: footprint Capacitor_Tantalum_SMD:CP_EIA-2012-12_Kemet-R_Pad1.30x1.05mm_HandSolder -> Capacitor_Tantalum_SMD:CP_EIA-3216-10_Kemet-I_Pad1.58x1.35mm_HandSolder; AliExpress (none) -> https://www.aliexpress.com/item/1005002349845549.html?spm=a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
- J1, JP1: AliExpress (none) -> https://www.aliexpress.com/item/32897706396.html?spm=a2g0o.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; Digikey (none) -> S1022E-02-ND
- J2: AliExpress (none) -> https://www.aliexpress.com/item/32897706396.html?spm=a2g0o.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; Digikey (none) -> S1222E-04-ND
- Q1, Q2, Q3, Q4, Q5: AliExpress (none) -> https://www.aliexpress.com/item/32844509358.html?spm=a2g0o.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; Digikey (none) -> BSS138CT-ND
- R1, R10, R11, R12, R2, R3, R4, R5, R6, R7, R8, R9: AliExpress (none) -> https://www.aliexpress.com/item/1005002384017954.html?spm=a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; Digikey (none) -> 2368-SR1-0603-610-ND
- U1: AliExpress (none) -> https://www.aliexpress.com/item/32791545218.html?spm=a2g0s.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; Digikey (none) -> ED3048-5-ND
- U2: AliExpress (none) -> https://www.aliexpress.com/item/32866552942.html?spm=a2g0o.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; Digikey (none) -> 1175-1490-ND
- U3: AliExpress (none) -> https://www.aliexpress.com/item/32537772545.html?spm=a2g0o.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; Digikey (none) -> 296-1602-5-ND
- U4: AliExpress (none) -> https://www.aliexpress.com/item/1005002119323721.html?spm=a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; Digikey (none) -> ESP-12SRF-ND
- U5: AliExpress (none) -> https://www.aliexpress.com/item/4001158893261.html?spm=a2g0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; Digikey (none) -> LM1117IMP-3.3/NOPBCT-ND
- Y1: AliExpress (none) -> https://www.aliexpress.com/item/32700741834.html?spm=a2g0o.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
